Commit message: Add joystick teleoperation and iPhone base tracking
Add fixed-speed chassis control, optional torso modes, homing guards, gripper contact handling, and updated collision geometry.

Include ARKit publisher and calibration tools, printable/editable phone mounts, and a pinned Record3D USB latency patch. Improve camera timing checks, recording provenance, native telemetry sidecars, and public setup documentation.

Clean up obsolete comments and unused code while preserving CLI and configuration behavior. Validation: 337 hardware-free tests passed, 3 mesh-dependent tests skipped; lint and formatting passed.

File: src/omniteleop/assets/vega_with_robotiq.urdf (robot description, URDF)
Before this commit: robot vega-1, 47 links, 46 joints
Links:
- added link L_fingertip_neg
- added link L_fingertip_pos
- added link L_gripper_connector
- added link L_wrist_cam_bracket
- added link L_wrist_camera
- added link L_wrist_zed_mini
- added link R_fingertip_neg
- added link R_fingertip_pos
- added link R_gripper_connector
- added link R_wrist_cam_bracket
- added link R_wrist_camera
- added link R_wrist_zed_mini
Joints:
- added joint L_fingertip_neg_j0: type fixed, parent L_robotiq, child L_fingertip_neg, origin xyz=-0.05636 0.00077 -0.08929 rpy=0 0 3.14159265
- added joint L_fingertip_pos_j0: type fixed, parent L_robotiq, child L_fingertip_pos, origin xyz=0.05636 -0.00008 -0.08929 rpy=0 0 0
- added joint L_gripper_connector_mount: type fixed, parent L_ee, child L_gripper_connector, origin xyz=0 0 -0.0029998 rpy=0 0 0, axis 0 0 0
- added joint L_wrist_cam_bracket_mount: type fixed, parent L_ee, child L_wrist_cam_bracket, origin xyz=-0.051883246545 0.000029548342 0.034751587884 rpy=-1.288710320044 0.000000000000 -1.570792653590, axis 0 0 0
- added joint L_wrist_camera_mount: type fixed, parent L_wrist_zed_mini, child L_wrist_camera, origin xyz=0.041094 0.041479 -0.017168 rpy=1.530991 0.032838 3.128694, axis 0 0 0
- added joint L_wrist_zed_mini_mount: type fixed, parent L_ee, child L_wrist_zed_mini, origin xyz=-0.086119536449 0.000029422585 0.041038557910 rpy=1.789077809687 0.000000000000 1.570800000000, axis 0 0 0
- added joint R_fingertip_neg_j0: type fixed, parent R_robotiq, child R_fingertip_neg, origin xyz=-0.05636 0.00077 -0.08929 rpy=0 0 3.14159265
- added joint R_fingertip_pos_j0: type fixed, parent R_robotiq, child R_fingertip_pos, origin xyz=0.05636 -0.00008 -0.08929 rpy=0 0 0
- added joint R_gripper_connector_mount: type fixed, parent R_ee, child R_gripper_connector, origin xyz=0 0 -0.0029998 rpy=0 0 0, axis 0 0 0
- added joint R_wrist_cam_bracket_mount: type fixed, parent R_ee, child R_wrist_cam_bracket, origin xyz=-0.051883246545 0.000029548342 0.034751587884 rpy=-1.288710320044 0.000000000000 -1.570792653590, axis 0 0 0
- added joint R_wrist_camera_mount: type fixed, parent R_wrist_zed_mini, child R_wrist_camera, origin xyz=0.028939 0.046335 0.005880 rpy=1.430370 0.015275 -3.126599, axis 0 0 0
- added joint R_wrist_zed_mini_mount: type fixed, parent R_ee, child R_wrist_zed_mini, origin xyz=-0.086119536449 0.000029422585 0.041038557910 rpy=1.789077809687 0.000000000000 1.570800000000, axis 0 0 0
- joint L_robotiq_j0: origin xyz=0 0 0.24 rpy=0 0 1.5708 -> xyz=0 0 0.2341892 rpy=0 0 1.5708
- joint R_robotiq_j0: origin xyz=0 0 0.24 rpy=0 0 1.5708 -> xyz=0 0 0.2341892 rpy=0 0 1.5708
